File: PCB_SMD/dmx_rgb.sch (KiCad schematic (older format))
At the start: 30 parts, among them J1 CONN_01X02, J2 Conn_02x04_Odd_Even, J3 Conn_02x03_Odd_Even, J4 CONN_01X03, J5 CONN_01X04, J6 CONN_01X04, Q1 Q_NMOS_GSD, Q2 Q_NMOS_GSD, Q3 Q_NMOS_GSD, U1 ATTINY2313-20PU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

Commit message: spannungs wandler getauscht
Parts:
- removed C6: CP, Capacitors_THT:CP_Radial_D5.0mm_P2.50mm, symbol CP
- removed C7: C, Resistors_SMD:R_0805_HandSoldering, symbol C
- removed U2: L7805, DPAK:DPAK, symbol L7805
- removed Y1: Crystal, Crystals:Crystal_SMD_SeikoEpson_MA505-2pin_12.7x5.1mm_HandSoldering, symbol Crystal
- added C6: CP, Capacitors_SMD:CP_Elec_4x5.8, symbol Device:CP
- added C7: C, Resistors_SMD:R_0805_HandSoldering, symbol Device:C
- added MH1, MH2, MH3: MountingHole, Mounting_Holes:MountingHole_2.2mm_M2, symbol Mechanical:MountingHole
- added U2: LM1117-3.3, TO_SOT_Packages_SMD:SOT-223-3Lead_TabPin2, symbol regul:LM1117-3.3
- added Y1: Crystal_GND24, Crystals:Crystal_SMD_EuroQuartz_MQ2-2pin_7.0x5.0mm_HandSoldering, symbol Device:Crystal_GND24
- C1, C2, C3, C4, C8: symbol C -> Device:C
- C5: symbol CP -> Device:CP
- D1: symbol D_Bridge_+A-A -> dmx_rgb-rescue:D_Bridge_+A-A
- J1: symbol Conn_01x02 -> conn:Conn_01x02
- J2: symbol Conn_02x04_Odd_Even -> conn:Conn_02x04_Odd_Even
- J3: symbol Conn_02x03_Odd_Even -> conn:Conn_02x03_Odd_Even
- J4: symbol Conn_01x03 -> conn:Conn_01x03
- J5, J6: symbol Conn_01x04 -> conn:Conn_01x04
- Q1, Q2, Q3: symbol Q_NMOS_GSD -> Device:Q_NMOS_GSD
- R1, R2, R3, R4, R5, R6, R7, R8: symbol R -> Device:R
- U1: symbol ATTINY2313-20PU -> atmel:ATTINY2313-20PU
- U3: symbol MAX485E -> dmx_rgb-rescue:MAX485E
Connections:
- wire segments 106 -> 137
Other:
- moved on the sheet: J2, J3, R1, R2, R4, R5

Commit message: node red mqtt json upgrade
Parts:
- C1, C2: value C -> 10p
- C3, C4, C7, C8: value C -> 100n
- Q1, Q2, Q3: value Q_NMOS_GSD -> IRLML 6244
- R1, R2, R3, R4, R5, R7, R8: value R -> 10k
- U1: value ATTINY2313-20PU -> ATTINY2313A-SU
- U2: value LM1117-3.3 -> LM1117 IMP-3.3
- U3: value MAX485E -> MAX3485 CSA
- Y1: value Crystal_GND24 -> 16,000000-MQ
Changed lines of the file:
@@
 P 1450 2650
 F 0 "C1" H 1475 2750 50  0000 L CNN
-F 1 "C" H 1475 2550 50  0000 L CNN
+F 1 "10p" H 1475 2550 50  0000 L CNN
 F 2 "Capacitors_SMD:C_0805_HandSoldering" H 1488 2500 50  0001 C CNN
 F 3 "" H 1450 2650 50  0001 C CNN
@@
 P 1450 2950
 F 0 "C2" H 1475 3050 50  0000 L CNN
-F 1 "C" H 1475 2850 50  0000 L CNN
+F 1 "10p" H 1475 2850 50  0000 L CNN
 F 2 "Capacitors_SMD:C_0805_HandSoldering" H 1488 2800 50  0001 C CNN
 F 3 "" H 1450 2950 50  0001 C CNN
@@
 P 1800 2400
 F 0 "C3" H 1825 2500 50  0000 L CNN
-F 1 "C" H 1825 2300 50  0000 L CNN
+F 1 "100n" H 1825 2300 50  0000 L CNN
 F 2 "Capacitors_SMD:C_0805_HandSoldering" H 1838 2250 50  0001 C CNN
 F 3 "" H 1800 2400 50  0001 C CNN
@@
 P 3000 2050
 F 0 "C4" H 3025 2150 50  0000 L CNN
-F 1 "C" H 3025 1950 50  0000 L CNN
+F 1 "100n" H 3025 1950 50  0000 L CNN
 F 2 "Capacitors_SMD:C_0805_HandSoldering" H 3038 1900 50  0001 C CNN
 F 3 "" H 3000 2050 50  0001 C CNN
@@
 P 2000 2200
 F 0 "R3" V 2080 2200 50  0000 C CNN
-F 1 "R" V 2000 2200 50  0000 C CNN
+F 1 "10k" V 2000 2200 50  0000 C CNN
 F 2 "Resistors_SMD:R_0805_HandSoldering" V 1930 2200 50  0001 C CNN
 F 3 "" H 2000 2200 50  0001 C CNN
@@
 P 5800 2200
 F 0 "C8" H 5825 2300 50  0000 L CNN
-F 1 "C" H 5825 2100 50  0000 L CNN
+F 1 "100n" H 5825 2100 50  0000 L CNN
 F 2 "Resistors_SMD:R_0805_HandSoldering" H 5838 2050 50  0001 C CNN
 F 3 "" H 5800 2200 50  0001 C CNN
@@
 P 2950 6000
 F 0 "R7" V 3030 6000 50  0000 C CNN
-F 1 "R" V 2950 6000 50  0000 C CNN
+F 1 "10k" V 2950 6000 50  0000 C CNN
 F 2 "Resistors_SMD:R_0805_HandSoldering" V 2880 6000 50  0001 C CNN
 F 3 "" H 2950 6000 50  0001 C CNN
@@
 P 4300 6000
 F 0 "R8" V 4380 6000 50  0000 C CNN
-F 1 "R" V 4300 6000 50  0000 C CNN
+F 1 "10k" V 4300 6000 50  0000 C CNN
 F 2 "Resistors_SMD:R_0805_HandSoldering" V 4230 6000 50  0001 C CNN
 F 3 "" H 4300 6000 50  0001 C CNN
@@
 P 1750 5800
 F 0 "Q1" H 1950 5850 50  0000 L CNN
-F 1 "Q_NMOS_GSD" H 1950 5750 50  0000 L CNN
+F 1 "IRLML 6244" H 1950 5750 50  0000 L CNN
 F 2 "TO_SOT_Packages_SMD:SOT-23" H 1950 5900 50  0001 C CNN
 F 3 "" H 1750 5800 50  0001 C CNN
@@
 P 3200 5800
 F 0 "Q2" H 3400 5850 50  0000 L CNN
-F 1 "Q_NMOS_GSD" H 3400 5750 50  0000 L CNN
+F 1 "IRLML 6244" H 3400 5750 50  0000 L CNN
 F 2 "TO_SOT_Packages_SMD:SOT-23" H 3400 5900 50  0001 C CNN
 F 3 "" H 3200 5800 50  0001 C CNN
@@
 P 4550 5800
 F 0 "Q3" H 4750 5850 50  0000 L CNN
-F 1 "Q_NMOS_GSD" H 4750 5750 50  0000 L CNN
+F 1 "IRLML 6244" H 4750 5750 50  0000 L CNN
 F 2 "TO_SOT_Packages_SMD:SOT-23" H 4750 5900 50  0001 C CNN
 F 3 "" H 4550 5800 50  0001 C CNN
@@
 P 9200 1400
 F 0 "R4" V 9280 1400 50  0000 C CNN
-F 1 "R" V 9200 1400 50  0000 C CNN
+F 1 "10k" V 9200 1400 50  0000 C CNN
 F 2 "Resistors_SMD:R_0805_HandSoldering" V 9130 1400 50  0001 C CNN
 F 3 "" H 9200 1400 50  0001 C CNN
@@
 P 9400 1500
 F 0 "R5" V 9480 1500 50  0000 C CNN
-F 1 "R" V 9400 1500 50  0000 C CNN
+F 1 "10k" V 9400 1500 50  0000 C CNN
 F 2 "Resistors_SMD:R_0805_HandSoldering" V 9330 1500 50  0001 C CNN
 F 3 "" H 9400 1500 50  0001 C CNN
@@
 P 7900 1400
 F 0 "R2" V 7980 1400 50  0000 C CNN
-F 1 "R" V 7900 1400 50  0000 C CNN
+F 1 "10k" V 7900 1400 50  0000 C CNN
 F 2 "Resistors_SMD:R_0805_HandSoldering" V 7830 1400 50  0001 C CNN
 F 3 "" H 7900 1400 50  0001 C CNN
@@
 P 7700 1500
 F 0 "R1" V 7780 1500 50  0000 C CNN
-F 1 "R" V 7700 1500 50  0000 C CNN
+F 1 "10k" V 7700 1500 50  0000 C CNN
 F 2 "Resistors_SMD:R_0805_HandSoldering" V 7630 1500 50  0001 C CNN
 F 3 "" H 7700 1500 50  0001 C CNN
@@
 P 3200 3200
 F 0 "U1" H 2250 4200 50  0000 C CNN
-F 1 "ATTINY2313-20PU" H 4000 2300 50  0000 C CNN
+F 1 "ATTINY2313A-SU" H 4000 2300 50  0000 C CNN
 F 2 "Housings_SOIC:SOIC-20W_7.5x12.8mm_Pitch1.27mm" H 3200 3200 50  0001 C CIN
 F 3 "" H 3200 3200 50  0001 C CNN
@@
 P 6000 2700
 F 0 "U3" H 5760 3150 50  0000 C CNN
-F 1 "MAX485E" H 6030 3150 50  0000 L CNN
+F 1 "MAX3485 CSA" H 6030 3150 50  0000 L CNN
 F 2 "Housings_SOIC:SO-8_5.3x6.2mm_Pitch1.27mm" H 6000 2000 50  0001 C CNN
 F 3 "" H 6000 2750 50  0001 C CNN
@@
 P 4800 950
 F 0 "U2" H 4800 1192 50  0000 C CNN
-F 1 "LM1117-3.3" H 4800 1101 50  0000 C CNN
+F 1 "LM1117 IMP-3.3" H 4800 1101 50  0000 C CNN
 F 2 "TO_SOT_Packages_SMD:SOT-223-3Lead_TabPin2" H 4800 950 50  0001 C CNN
 F 3 "http://www.ti.com/lit/ds/symlink/lm1117.pdf" H 4800 950 50  0001 C CNN
@@
 P 5150 1150
 F 0 "C7" H 5175 1250 50  0000 L CNN
-F 1 "C" H 5175 1050 50  0000 L CNN
+F 1 "100n" H 5175 1050 50  0000 L CNN
 F 2 "Resistors_SMD:R_0805_HandSoldering" H 5188 1000 50  0001 C CNN
 F 3 "" H 5150 1150 50  0001 C CNN
@@
 P 1800 2800
 F 0 "Y1" V 1754 3041 50  0000 L CNN
-F 1 "Crystal_GND24" V 1845 3041 50  0000 L CNN
+F 1 "16,000000-MQ" V 1845 3041 50  0000 L CNN
 F 2 "Crystals:Crystal_SMD_EuroQuartz_MQ2-2pin_7.0x5.0mm_HandSoldering" H 1800 2800 50  0001 C CNN
 F 3 "~" H 1800 2800 50  0001 C CNN
